Commit message: renamed disk_joint to motor_joint (fixed bug)

File: qube_bringup/urdf/controlled_qube.urdf.xacro (robot description, xacro)
@@ -1,4 +1,4 @@
 <?xml version="1.0"?>
-<robot xmlns:xacro="http://www.ros.org/wiki/xacro" name="robot_name">
+<robot xmlns:xacro="http://www.ros.org/wiki/xacro" name="qube_scene">
 <xacro:arg name="baud_rate" default="115200"/> <!--Communication baud rate of Arduino-->
 <xacro:arg name="device" default="none"/> <!--Name of USB device-->
@@ -6,8 +6,16 @@
 <xacro:include filename="$(find qube_driver)/ros2_control/qube_driver.ros2_control.xacro"/>
 <xacro:qube_driver_ros2_control
-    name="qube"
-    prefix=""
+    name="qube_driver"
+    prefix="qube_"
     baud_rate="$(arg baud_rate)"
     device="$(arg device)"
-    simulation="$(arg simulation)"/>
+    simulation="$(arg simulation)"/> <!--prefix for driver must be the same as for qube macro-->
+<xacro:include filename="$(find qube_description)/urdf/qube.macro.xacro"/>
+<xacro:qube prefix="qube_"/>
+<link name="world"/>
+<joint name="world_to_base" type="fixed">
+<parent link="world"/>
+<child link="qube_base_link"/>
+<origin xyz="0 0 0" rpy="0 0 0"/>
+</joint>
 </robot>

File: qube_description/urdf/qube.macro.xacro (robot description, xacro)
@@ -52,5 +52,5 @@
       <origin xyz="0 0 ${box_z/2}"/>
     </joint>
-    <joint name="${prefix}disk_joint" type="revolute">
+    <joint name="${prefix}motor_joint" type="revolute">
       <parent link="${prefix}body_link"/>
       <child link="${prefix}disk_link"/>

Commit message: EVERYTHING WORKS

File: qube_bringup/urdf/controlled_qube.urdf.xacro (robot description, xacro)
@@ -3,18 +3,18 @@
 <xacro:arg name="baud_rate" default="115200"/> <!--Communication baud rate of Arduino-->
 <xacro:arg name="device" default="none"/> <!--Name of USB device-->
-<xacro:arg name="simulation" default="true"/> <!--Whether this should be run as a simulation-->
+<xacro:arg name="simulation" default="false"/> <!--Whether this should be run as a simulation-->
 <xacro:include filename="$(find qube_driver)/ros2_control/qube_driver.ros2_control.xacro"/>
 <xacro:qube_driver_ros2_control
-    name="qube_driver"
-    prefix="qube_"
+    name="driver_"
+    prefix=""
     baud_rate="$(arg baud_rate)"
     device="$(arg device)"
     simulation="$(arg simulation)"/> <!--prefix for driver must be the same as for qube macro-->
 <xacro:include filename="$(find qube_description)/urdf/qube.macro.xacro"/>
-<xacro:qube prefix="qube_"/>
+<xacro:qube prefix=""/>
 <link name="world"/>
 <joint name="world_to_base" type="fixed">
 <parent link="world"/>
-<child link="qube_base_link"/>
+<child link="base_link"/>
 <origin xyz="0 0 0" rpy="0 0 0"/>
 </joint>

File: qube_description/urdf/qube.macro.xacro (robot description, xacro)
@@ -56,5 +56,5 @@
       <child link="${prefix}disk_link"/>
       <origin xyz="0 0 ${box_z/2 + disk_length/2}"/>
-      <axis xyz="0 0 1"/>
+      <axis xyz="0 0 -1"/>
       <limit lower="-1.5708" upper="1.5708" effort="100" velocity="100"/>
     </joint>

Commit message: docs

File: qube_bringup/urdf/controlled_qube.urdf.xacro (robot description, xacro)
@@ -10,11 +10,11 @@
     baud_rate="$(arg baud_rate)"
     device="$(arg device)"
-    simulation="$(arg simulation)"/> <!--prefix for driver must be the same as for qube macro-->
+    simulation="$(arg simulation)"/>
 <xacro:include filename="$(find qube_description)/urdf/qube.macro.xacro"/>
-<xacro:qube prefix=""/>
+<xacro:qube prefix=""/> <!--prefix for qube macro must be the same as for qube_driver-->
 <link name="world"/>
 <joint name="world_to_base" type="fixed">
 <parent link="world"/>
-<child link="base_link"/>
+<child link="base_link"/> <!--Prefix of this must match Qube macro prefix-->
 <origin xyz="0 0 0" rpy="0 0 0"/>
 </joint>

Commit message: docs

File: qube_bringup/urdf/controlled_qube.urdf.xacro (robot description, xacro)
@@ -12,9 +12,9 @@
     simulation="$(arg simulation)"/>
 <xacro:include filename="$(find qube_description)/urdf/qube.macro.xacro"/>
-<xacro:qube prefix=""/> <!--prefix for qube macro must be the same as for qube_driver-->
+<xacro:qube prefix=""/> <!--Prefix of this must match Qube macro prefix-->
 <link name="world"/>
 <joint name="world_to_base" type="fixed">
 <parent link="world"/>
-<child link="base_link"/> <!--Prefix of this must match Qube macro prefix-->
+<child link="base_link"/>
 <origin xyz="0 0 0" rpy="0 0 0"/>
 </joint>
